File: TVC99.kicad_sch (KiCad schematic)
At the start: 19 parts, among them J1 Conn_01x24_Pin, J2 Conn_01x24_Pin, J5 Ground, J6 PWM DC motor control, M1 Motor_Servo, M2 Motor_Servo, M3 Motor_Servo, Q1 IRLB8721PBF, Q2 IRLB8721PBF, U1 Teensy4.1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

Commit message: docs: pcb files
Parts:
- BZ1: footprint (none) -> Buzzer_Beeper:Buzzer_TDK_PS1240P02BT_D12.2mm_H6.5mm
- J6: footprint (none) -> Connector_JST:JST_XH_B3B-XH-AM_1x03_P2.50mm_Vertical
- M1: renamed from M3; footprint (none) -> Connector_JST:JST_XH_B3B-XH-AM_1x03_P2.50mm_Vertical
- M2: renamed from M1; footprint (none) -> Connector_JST:JST_XH_B3B-XH-AM_1x03_P2.50mm_Vertical
- M3: renamed from M2; footprint (none) -> Connector_JST:JST_XH_B3B-XH-AM_1x03_P2.50mm_Vertical
- U1: footprint Teensy_footprints:Teensy41 -> Teensy4.1:Teensy41
- U3: renamed from U2; footprint (none) -> LoRa_RF95:LoRa_RF95 Breakout
- U5: renamed from U6; footprint (none) -> BNO055:BNO055
- renumbered U4 to U2, U5 to U4, U3 to U6
Connections:
- net at J1.12 (Pin_12), U1.12 (10_CS_MQSR): now also U3.14 (CS); no longer U3.13 (MOSI), U6.7 (CS)
- net at J1.13 (Pin_13), U1.13 (11_MOSI_CTX1): now also U3.13 (MOSI), U6.7 (CS); no longer U3.12 (MISO), U6.6 (MOSI)
- net at J1.14 (Pin_14), U1.14 (12_MISO_MQSL): now also U3.12 (MISO), U6.6 (MOSI); no longer U3.11 (SCK), U6.5 (MISO)
- net at J1.2 (Pin_2), U1.2 (0_RX1_CRX2_CS1): no longer U3.14 (CS)
- net at J2.11 (Pin_11), U1.35 (13_SCK_LED): now also U3.11 (SCK), U6.5 (MISO)
- net at J2.23 (Pin_23), U1.47 (GND), U3.8 (GND)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: now also U5.7 (GND), U7.7 (GND)
